File: Eagle/quad_copter.brd (EAGLE design)
At the start: 99 x 105.1 mm, 13 parts, among them X1 STM32F4_DISC

Commit message: Screenshots
Routing:
- net 0V: track 221.4 -> 239.2 mm, vias 8 -> 6
Other:
- board size 99 x 105.1 mm -> 97.8 x 105.1 mm
Changed lines of the file:
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@@
 <layer number="20" name="Dimension" color="15" fill="1" visible="yes" active="yes"/>
 <layer number="21" name="tPlace" color="7" fill="1" visible="yes" active="yes"/>
-<layer number="22" name="bPlace" color="7" fill="1" visible="yes" active="yes"/>
+<layer number="22" name="bPlace" color="7" fill="1" visible="no" active="yes"/>
 <layer number="23" name="tOrigins" color="15" fill="1" visible="yes" active="yes"/>
 <layer number="24" name="bOrigins" color="15" fill="1" visible="no" active="yes"/>
-<layer number="25" name="tNames" color="7" fill="1" visible="no" active="yes"/>
+<layer number="25" name="tNames" color="7" fill="1" visible="yes" active="yes"/>
 <layer number="26" name="bNames" color="7" fill="1" visible="no" active="yes"/>
 <layer number="27" name="tValues" color="7" fill="1" visible="no" active="yes"/>
@@
 <plain>
 <wire x1="0" y1="0" x2="97.77" y2="0" width="0" layer="20"/>
-<wire x1="97.77" y1="0" x2="96.5" y2="105.08" width="0" layer="20"/>
-<wire x1="96.5" y1="105.08" x2="-1.27" y2="105.08" width="0" layer="20"/>
-<wire x1="-1.27" y1="105.08" x2="0" y2="0" width="0" layer="20"/>
+<wire x1="97.77" y1="0" x2="97.77" y2="105.08" width="0" layer="20"/>
+<wire x1="97.77" y1="105.08" x2="0" y2="105.08" width="0" layer="20"/>
+<wire x1="0" y1="105.08" x2="0" y2="0" width="0" layer="20"/>
 </plain>
 <attributes>
@@
 <wire x1="13.97" y1="48.26" x2="7.62" y2="48.26" width="1.4224" layer="16"/>
 <wire x1="7.62" y1="48.26" x2="7.62" y2="55.88" width="1.4224" layer="16"/>
-<wire x1="7.62" y1="55.88" x2="13.97" y2="55.88" width="1.4224" layer="16"/>
-<wire x1="13.97" y1="55.88" x2="13.97" y2="72.39" width="1.4224" layer="16"/>
-<via x="13.97" y="72.39" extent="1-16" drill="0.6" diameter="2.1844" shape="square"/>
-<wire x1="13.97" y1="72.39" x2="13.97" y2="73.66" width="1.4224" layer="1"/>
-<wire x1="13.97" y1="73.66" x2="82.55" y2="73.66" width="1.4224" layer="1"/>
+<wire x1="7.62" y1="55.88" x2="11.43" y2="55.88" width="1.4224" layer="16"/>
+<wire x1="11.43" y1="55.88" x2="11.43" y2="72.39" width="1.4224" layer="16"/>
+<via x="11.43" y="72.39" extent="1-16" drill="0.6" diameter="2.1844" shape="square"/>
+<wire x1="11.43" y1="72.39" x2="11.43" y2="73.66" width="1.4224" layer="1"/>
+<wire x1="11.43" y1="73.66" x2="82.55" y2="73.66" width="1.4224" layer="1"/>
 <wire x1="82.55" y1="73.66" x2="82.55" y2="71.12" width="1.4224" layer="1"/>
 <via x="82.55" y="71.12" extent="1-16" drill="0.6" diameter="2.1844" shape="square"/>
@@
 <wire x1="55.88" y1="1.27" x2="40.64" y2="1.27" width="1.4224" layer="16"/>
 <wire x1="40.64" y1="1.27" x2="40.64" y2="2.54" width="1.4224" layer="16"/>
-<wire x1="22.86" y1="68.58" x2="19.05" y2="68.58" width="1.4224" layer="16"/>
-<via x="19.05" y="68.58" extent="1-16" drill="0.6" diameter="2.1844" shape="square"/>
-<wire x1="19.05" y1="68.58" x2="5.08" y2="68.58" width="1.4224" layer="1"/>
-<via x="5.08" y="68.58" extent="1-16" drill="0.6" diameter="2.1844" shape="square"/>
-<wire x1="5.08" y1="68.58" x2="5.08" y2="48.26" width="1.4224" layer="16"/>
+<wire x1="5.08" y1="77.47" x2="5.08" y2="48.26" width="1.4224" layer="16"/>
 <wire x1="40.64" y1="2.54" x2="27.94" y2="10.16" width="1.27" layer="1"/>
 <wire x1="55.88" y1="2.54" x2="68.58" y2="10.16" width="1.27" layer="1"/>
+<wire x1="22.86" y1="68.58" x2="17.78" y2="68.58" width="1.4224" layer="16"/>
+<wire x1="17.78" y1="68.58" x2="17.78" y2="77.47" width="1.4224" layer="16"/>
+<wire x1="17.78" y1="77.47" x2="5.08" y2="77.47" width="1.4224" layer="16"/>
 </signal>
 <signal name="N$3">
